File: power.sch (KiCad schematic (older format))
At the start: 52 parts, among them J2 USB_C_Receptacle_USB2.0, Q1 FS8205A, Q6 2N7002, Q7 AO3401A, Q8 2N7002, U3 SY7088, U4 XC6206P332MR, U5 DW01+G, U6 TP4056, U9 BQ34Z100

Commit message: Reduce paste coverage on QFN and DFN thermal pads
Parts:
- U3: footprint Package_DFN_QFN:DFN-8-1EP_3x2mm_P0.5mm_EP1.3x1.5mm -> DFN_little_paste:DFN-8-1EP_3x2mm_P0.5mm_EP1.3x1.5mm_little_paste
Changed lines of the file:
@@
 F 0 "U3" H 7250 4315 50  0000 C CNN
 F 1 "SY7088" H 7250 4224 50  0000 C CNN
-F 2 "Package_DFN_QFN:DFN-8-1EP_3x2mm_P0.5mm_EP1.3x1.5mm" H 7250 3850 50  0001 C CNN
+F 2 "DFN_little_paste:DFN-8-1EP_3x2mm_P0.5mm_EP1.3x1.5mm_little_paste" H 7250 3850 50  0001 C CNN
 F 3 "https://datasheet.lcsc.com/szlcsc/Silergy-Corp-SY7088DGC_C178240.pdf" H 7250 3850 50  0001 C CNN
 F 4 "C178240" H 7250 3850 50  0001 C CNN "LCSC"
